Commit message: Update A

File: Minichallenges/minichal1/include/puzzlebot_jetson_ed_urdf.urdf (robot description, URDF)
Before this commit: robot Puzzlebot Jetson-Lidar Ed., 2 links, 1 joints
Links:
- added link right_wheel, mass 0.01; collision mesh filename=package://minichal1/robot_models/MCR2_1000_13_Chassis.stl; visual mesh filename=package://minichal1/robot_models/MCR2_1000_13_Chassis.stl
- link chassis: geometry collision mesh filename=package://minichal1/robot_models/MCR2_1000_13_Chassis.stl; visual mesh filename=package://minichal1/robot_models/MCR2_1000_13_Chassis.stl
Joints:
- added joint right_wheel_joint: type continuous, parent chassis, child right_wheel, origin xyz=0.0 0.0 0.05

Commit message: Update add

File: Minichallenges/minichal1/include/puzzlebot_jetson_ed_urdf.urdf (robot description, URDF)
Before this commit: robot Puzzlebot Jetson-Lidar Ed., 2 links, 1 joints
Links:
- link chassis: geometry collision mesh filename=/robot_models/MCR2_1000_13_Chassis.stl; visual mesh filename=/robot_models/MCR2_1000_13_Chassis.stl

Commit message: minichal1

File: Minichallenges/minichal1/include/puzzlebot_jetson_ed_urdf.urdf (robot description, URDF)
Before this commit: robot Puzzlebot Jetson-Lidar Ed., 2 links, 1 joints
Links:
- added link left_wheel, mass 0.01; collision mesh filename=package://minichal1/robot_models/MCR2_1000_1_1_Wheel_Couple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; visual mesh filename=package://minichal1/robot_models/MCR2_1000_1_1_Wheel_Couple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
- added link right_wheel, mass 0.01; collision mesh filename=package://minichal1/robot_models/MCR2_1000_1_1_Wheel_Couple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; visual mesh filename=package://minichal1/robot_models/MCR2_1000_1_1_Wheel_Couple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
- link chassis: geometry collision mesh filename=package://minichal1/robot_models/MCR2_1000_13_Chassis.stl; visual mesh filename=package://minichal1/robot_models/MCR2_1000_13_Chassis.stl
Joints:
- added joint wl_joint: type continuous, parent base_link, child left_wheel, origin xyz=0.0 0.0 0.05, axis 0 1 0
- added joint wr_joint: type continuous, parent base_link, child right_wheel, origin xyz=0.0 0.0 0.05, axis 0 1 0

Commit message: Arreglos

File: Minichallenges/minichal1/include/puzzlebot_jetson_ed_urdf.urdf (robot description, URDF)
Before this commit: robot Puzzlebot Jetson-Lidar Ed., 4 links, 3 joints
Joints:
- joint wl_joint: parent base_link -> chassis
- joint wr_joint: parent base_link -> chassis

Commit message: Fixed launch

File: Minichallenges/minichal1/include/puzzlebot_jetson_ed_urdf.urdf (robot description, URDF)
Before this commit: robot Puzzlebot Jetson-Lidar Ed., 4 links, 3 joints
Links:
- added link ref_l
- added link ref_r
Joints:
- added joint wl_joint_ref: type fixed, parent chassis, child ref_l, origin xyz=0.0 0.0 0.05
- added joint wr_joint_ref: type fixed, parent chassis, child ref_r, origin xyz=0.0 0.0 0.05
- joint wl_joint: origin xyz=0.0 0.0 0.05 -> xyz=0.0 0.0 0.0
- joint wr_joint: origin xyz=0.0 0.0 0.05 -> xyz=0.0 0.0 0.0; parent chassis -> ref_r

Commit message: movimiento llanta

File: Minichallenges/minichal1/include/puzzlebot_jetson_ed_urdf.urdf (robot description, URDF)
Before this commit: robot Puzzlebot Jetson-Lidar Ed., 6 links, 5 joints
Links:
- removed link ref_l
- removed link ref_r
