Commit message: Package rename. Dont forget to do a catkin_make

File: Minichallenges/minichal2/include/puzzlebot_2.urdf (robot description, URDF)
Before this commit: robot Puzzlebot, 4 links, 3 joints
Links:
- link chassis: geometry collision mesh filename=package://minichal2/robot_models/MCR2_1000_13_Chassis.stl; visual mesh filename=package://minichal2/robot_models/MCR2_1000_13_Chassis.stl
- link left_wheel: geometry collision mesh filename=package://minichal2/robot_models/MCR2_1000_1_1_Wheel_Couple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; visual mesh filename=package://minichal2/robot_models/MCR2_1000_1_1_Wheel_Couple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
- link right_wheel: geometry collision mesh filename=package://minichal2/robot_models/MCR2_1000_1_1_Wheel_Couple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; visual mesh filename=package://minichal2/robot_models/MCR2_1000_1_1_Wheel_Couple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

File: Minichallenges/minichal2/include/puzzlebot_jetson_ed_urdf.urdf (robot description, URDF)
Before this commit: robot Puzzlebot Jetson-Lidar Ed., 3 links, 2 joints
Links:
- link chassis: geometry collision mesh filename=package://minichal2/robot_models/MCR2_1000_13_Chassis.stl; visual mesh filename=package://minichal2/robot_models/MCR2_1000_13_Chassis.stl
- link right_wheel: geometry collision mesh filename=package://minichal2/robot_models/MCR2_1000_13_Chassis.stl; visual mesh filename=package://minichal2/robot_models/MCR2_1000_13_Chassis.stl
