Commit message: Change the name of the package

File: Minichallenges/minichal4/include/puzzlebot_2.urdf (robot description, URDF)
Before this commit: robot Puzzlebot, 4 links, 3 joints
Links:
- link chassis: geometry collision mesh filename=package://minichal4/robot_models/MCR2_1000_13_Chassis.stl; visual mesh filename=package://minichal4/robot_models/MCR2_1000_13_Chassis.stl
- link left_wheel: geometry collision mesh filename=package://minichal4/robot_models/MCR2_1000_1_1_Wheel_Couple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; visual mesh filename=package://minichal4/robot_models/MCR2_1000_1_1_Wheel_Couple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
- link right_wheel: geometry collision mesh filename=package://minichal4/robot_models/MCR2_1000_1_1_Wheel_Couple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; visual mesh filename=package://minichal4/robot_models/MCR2_1000_1_1_Wheel_Couple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
